Commit message: add launch script, spawn not visible in gazebo

File: tmk_description/urdf/kitchen.urdf.xacro (robot description, xacro)
@@ -1,6 +1,8 @@
 <?xml version="1.0"?>
-<robot name="open_manipulator_p" xmlns:xacro="http://www.ros.org/wiki/xacro">
+<robot name="thormang" xmlns:xacro="http://www.ros.org/wiki/xacro">
   <!-- Import Rviz colors -->
-  <xacro:include filename="$(find open_manipulator_p_description)/urdf/materials.xacro"/>
+  <xacro:include filename="$(find tmk_description)/urdf/materials.xacro"/>
+  <gazebo reference="world"/>
+  <gazebo reference="kitchen_link"/>
   <!-- World with kitchen-->
   <link name="world"/>
@@ -14,5 +16,5 @@
       <origin xyz="0.0 0.0 0.0" rpy="0 0 0" />
       <geometry>
-        <mesh filename="package://open_manipulator_p_description/meshes/kitchen.stl"/>
+        <mesh filename="package://tmk_description/meshes/kitchen.stl"/>
       </geometry>
     </visual>
@@ -20,5 +22,5 @@
       <origin xyz="0.0 0.0 0.0" rpy="0 0 0" />
       <geometry>
-        <mesh filename="package://open_manipulator_p_description/meshes/kitchen_simple.stl"/>
+        <mesh filename="package://tmk_description/meshes/kitchen_simple.stl"/>
       </geometry>
     </collision>
